File: PocketBeagle.sch (KiCad schematic (older format))
At the start: 50 parts, among them SW1 POWER, U1 OSD3358-512M-BSM, U2 SN74LVC1G07DCK, U3 TPD4S012DRY, X1 10118192-0001LF, X2 MICROSD, Y1 24 MHz

Commit message: Pretty up the schematic and OSD component a bit
Signed-off-by: Michael Welling <mwelling@ieee.org>
Other:
- note removed: "Prototyped by: GHI Electronics, LLC"
- moved on the sheet: C2, C3, C4, C5, C6, C7, FB1, FB2, P1, P2, R10, R11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
