File: KiCAD/PocketBeagle.sch (KiCad schematic (older format))
At the start: 50 parts, among them SW1 POWER, U1 OSD3358-512M-BSM, U2 SN74LVC1G07DCK, U3 TPD4S012DRY, X1 10118192-0001LF, X2 MICROSD, Y1 24 MHz

Commit message: Sanitized schematic.
Removed "Pin not connected" errors. Net labels terminate on wire endpoints. Fixed P1 P2 symbol pin number overlap. Added sch heading
Connections:
- wire segments 475 -> 581
- no-connect marks 4 -> 54
Other:
- note added: "Pocket Beagle\n"
- note added: "https://beagleboard.org/pocket"
- moved on the sheet: P1
